Commit message: some dev before merge with Alex

File: FlexivPy/assets/r10s_with_capsules.urdf (robot description, URDF)
Before this commit: robot rizon10s, 10 links, 9 joints
Links:
- added link gripper, mass .9; visual cylinder length=.1 radius=.05
- added link gripper_c; collision sphere radius=0.02; collision sphere radius=0.02
Joints:
- added joint gripper_c_j: type fixed, parent gripper, child gripper_c, origin xyz=0 0 .10 rpy=0. 0 0.
- added joint gripper_j: type fixed, parent flange, child gripper, origin xyz=0 0 0 rpy=0. 0 0.
