Commit message: last commit before another merge!

File: FlexivPy/assets/flexiv_rizon10s_kinematics_w_gripper_mass.urdf (robot description, URDF)
Before this commit: robot rizon10s, 9 links, 8 joints
Links:
- added link tcp
Joints:
- added joint flange_to_tcp: type fixed, parent flange, child tcp, origin xyz=0.0 0.0 0.2 rpy=0.0 0.0 0.0

Commit message: add collision shapes to the w_gripper_mass

File: FlexivPy/assets/flexiv_rizon10s_kinematics_w_gripper_mass.urdf (robot description, URDF)
Before this commit: robot rizon10s, 10 links, 9 joints
Links:
- added link table; collision box size=2 2 .2; visual box size=2 2 .2
- added link wall; collision box size=.2 2 2; visual box size=.2 2 2
- link base_link: geometry collision cylinder length=0.10862981656370363 radius=0.10828695195085732; visual mesh filename=rizon10s/visual/v_link0.obj
- link flange: geometry collision cylinder length=0.15 radius=0.05
- link link1: geometry collision cylinder length=0.1820172995965973 radius=0.11; visual mesh filename=rizon10s/visual/v_link1.obj
- link link2: geometry collision cylinder length=0.1493152186350586 radius=0.09838617557444361; visual mesh filename=rizon10s/visual/v_link2.obj
- link link3: geometry collision cylinder length=0.17962829931741664 radius=0.08133934809468238; visual mesh filename=rizon10s/visual/v_link3.obj
- link link4: geometry collision cylinder length=0.14050029766613556 radius=0.08058945288499701; visual mesh filename=rizon10s/visual/v_link4.obj
- link link5: geometry collision cylinder length=0.1586607128833286 radius=0.06321103718614053; visual mesh filename=rizon10s/visual/v_link5.obj
- link link6: geometry collision cylinder length=0.1132427653650164 radius=0.07271170783548435; visual mesh filename=rizon10s/visual/v_link6.obj
- link link7: geometry collision cylinder length=0.08200182317353522 radius=0.05225879509988878; visual mesh filename=rizon10s/visual/v_link7.obj
Joints:
- added joint table_j: type fixed, parent base_link, child table, origin xyz=0 0 -0.11 rpy=0. 0 0.
- added joint wall_j: type fixed, parent base_link, child wall, origin xyz=-.4 0 0 rpy=0. 0 0.

Commit message: correction gripper state

File: FlexivPy/assets/flexiv_rizon10s_kinematics_w_gripper_mass.urdf (robot description, URDF)
Before this commit: robot rizon10s, 12 links, 11 joints
Links:
- link flange: geometry collision cylinder length=0.095 radius=0.05
